File: HAT_RPI_PnP.kicad_sch (KiCad schematic)
At the start: 5 parts, among them J14 Conn_02x20_Odd_Even

Commit message: rel 0.1
Parts:
- H1, H2, H3, H4: footprint Symbol:Screw_Generic_2.0x3.0mm_SilkScreen -> MountingHole:MountingHole_3.2mm_M3
Connections:
- net AUX1: now also J14.40 (Pin_40); no longer J14.8 (Pin_8)
- net AUX2: now also J14.38 (Pin_38); no longer J14.10 (Pin_10)
- net AUX3: now also J14.36 (Pin_36); no longer J14.12 (Pin_12)
- net AUX4: now also J14.32 (Pin_32); no longer J14.16 (Pin_16)
- net AUX5: now also J14.28 (Pin_28); no longer J14.18 (Pin_18)
- net AUX6: now also J14.26 (Pin_26); no longer J14.22 (Pin_22)
- net DIR_A: now also J14.29 (Pin_29); no longer J14.26 (Pin_26)
- net DIR_B: now also J14.23 (Pin_23); no longer J14.32 (Pin_32)
- net DIR_C: now also J14.17 (Pin_17); no longer J14.38 (Pin_38)
- net ENABLE: now also J14.19 (Pin_19); no longer J14.40 (Pin_40)
- net ENDSTOP1: now also J14.35 (Pin_35); no longer J14.31 (Pin_31)
- net ENDSTOP2: now also J14.37 (Pin_37); no longer J14.33 (Pin_33)
- net ENDSTOP3: now also J14.31 (Pin_31); no longer J14.35 (Pin_35)
- net ENDSTOP4: now also J14.33 (Pin_33); no longer J14.37 (Pin_37)
- net ISO_IN1: now also J14.18 (Pin_18); no longer J14.15 (Pin_15)
- net ISO_IN2: now also J14.13 (Pin_13); no longer J14.17 (Pin_17)
- net ISO_IN3: now also J14.16 (Pin_16); no longer J14.19 (Pin_19)
- net ISO_IN4: now also J14.11 (Pin_11); no longer J14.21 (Pin_21)
- net OUT1: now also J14.12 (Pin_12); no longer J14.23 (Pin_23)
- net OUT2: now also J14.10 (Pin_10); no longer J14.27 (Pin_27)
- net OUT3: now also J14.8 (Pin_8); no longer J14.29 (Pin_29)
- net STEP_A: now also J14.27 (Pin_27); no longer J14.24 (Pin_24)
- net STEP_B: now also J14.21 (Pin_21); no longer J14.28 (Pin_28)
- net STEP_C: now also J14.15 (Pin_15); no longer J14.36 (Pin_36)
- no-connect marks 5 -> 3
