File: Power.kicad_sch (KiCad schematic)
At the start: 20 parts, among them J12 Screw_Terminal_01x03, J9 Screw_Terminal_01x02, U7 TPS5430DDA

Commit message: rel 0.1
Connections:
- net +24V: now also J12.2 (Pin_2); no longer J12.1 (Pin_1)
- net +5V: now also J12.3 (Pin_3); no longer J12.2 (Pin_2)
- net GND: now also J12.1 (Pin_1); no longer J12.3 (Pin_3)
Changed lines of the file:
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@@
 	(symbol
 		(lib_id "power:+3.3V")
-		(at 187.96 163.83 90)
+		(at 187.96 166.37 90)
 		(unit 1)
 		(exclude_from_sim no)
@@
 		(fields_autoplaced yes)
 		(property "Reference" "#PWR0120"
-			(at 191.77 163.83 0)
+			(at 191.77 166.37 0)
 			(effects
 				(font
@@
 		)
 		(property "Value" "+24V"
-			(at 184.15 163.8299 90)
+			(at 184.15 166.3699 90)
 			(effects
 				(font
@@
 		)
 		(property "Footprint" ""
-			(at 187.96 163.83 0)
+			(at 187.96 166.37 0)
 			(effects
 				(font
@@
 		)
 		(property "Datasheet" ""
-			(at 187.96 163.83 0)
+			(at 187.96 166.37 0)
 			(effects
 				(font
@@
 		)
 		(property "Description" ""
-			(at 187.96 163.83 0)
+			(at 187.96 166.37 0)
 			(effects
 				(font
@@
 		(lib_id "Connector:Screw_Terminal_01x03")
 		(at 195.58 166.37 0)
-		(unit 1)
-		(exclude_from_sim no)
-		(in_bom yes)
-		(on_board yes)
-		(dnp no)
-		(fields_autoplaced yes)
+		(mirror x)
+		(unit 1)
+		(exclude_from_sim no)
+		(in_bom yes)
+		(on_board yes)
+		(dnp no)
 		(property "Reference" "J12"
-			(at 198.12 165.0999 0)
+			(at 198.12 167.6401 0)
 			(effects
 				(font
@@
 		)
 		(property "Value" "Screw_Terminal_01x03"
-			(at 198.12 167.6399 0)
+			(at 198.12 165.1001 0)
 			(effects
 				(font
@@
 		)
 		(instances
-			(project ""
+			(project "HAT_RPI_PnP"
 				(path "/5f6a39c5-abaf-4c77-9d7f-0c5e40ba26bf/71fc1cdf-affb-4c26-9c39-e444edbe6298"
 					(reference "J12")
@@
 	(symbol
 		(lib_id "power:+3.3V")
-		(at 187.96 166.37 90)
+		(at 187.96 163.83 90)
 		(unit 1)
 		(exclude_from_sim no)
@@
 		(fields_autoplaced yes)
 		(property "Reference" "#PWR0119"
-			(at 191.77 166.37 0)
+			(at 191.77 163.83 0)
 			(effects
 				(font
@@
 		)
 		(property "Value" "+5V"
-			(at 184.15 166.3699 90)
+			(at 184.15 163.8299 90)
 			(effects
 				(font
@@
 		)
 		(property "Footprint" ""
-			(at 187.96 166.37 0)
+			(at 187.96 163.83 0)
 			(effects
 				(font
@@
 		)
 		(property "Datasheet" ""
-			(at 187.96 166.37 0)
+			(at 187.96 163.83 0)
 			(effects
 				(font
@@
 		)
 		(property "Description" "Power symbol creates a global label with name \"+3.3V\""
-			(at 187.96 166.37 0)
-			(effects
-				(font
+			(at 187.96 163.83 0)
+			(effects
+				(font
